Commit message: spring kind of works

File: ezgripper_driver/urdf/ezgripper_dual.urdf.xacro (robot description, xacro)
@@ -18,4 +18,5 @@
       </collision>
     <inertial>
+      <origin xyz="0 0 0" rpy="0 0 0"/>
       <mass value=".3"/>
       <inertia ixx="0.01" ixy="0.0" ixz="0.0" iyy="0.01" iyz="0.0" izz="0.01"/>
@@ -52,4 +53,5 @@
       </collision>
       <inertial>
+        <origin xyz="-0.064 0 0.00132" rpy="0 0 0"/>
         <mass value=".025"/>
         <inertia ixx="0.01" ixy="0.0" ixz="0.0" iyy="0.01" iyz="0.0" izz="0.01"/>
@@ -94,3 +96,17 @@
    </plugin>
 </gazebo>
+<gazebo reference="only_ezgripper_knuckle_1">
+    <stopCfm>0.8</stopCfm>
+    <stopErp>100</stopErp>
+    <provideFeedback>true</provideFeedback>
+    <implicitSpringDamper>true</implicitSpringDamper>
+    <fudgeFactor>0.2</fudgeFactor>
+</gazebo>
+<gazebo reference="only_ezgripper_knuckle_2">
+    <stopCfm>0.8</stopCfm>
+    <stopErp>100</stopErp>
+    <provideFeedback>true</provideFeedback>
+    <implicitSpringDamper>true</implicitSpringDamper>
+    <fudgeFactor>0.2</fudgeFactor>
+</gazebo>
 </robot>

File: ezgripper_driver/urdf/ezgripper_dual_standalone.urdf.xacro (robot description, xacro)
@@ -6,6 +6,6 @@
 <xacro:include filename="$(find ezgripper_driver)/urdf/ezgripper_dual.urdf.xacro"/>
 <!-- Add the gripper -->
-<ezgripper_dual parent_link="base_link">
-<origin xyz="${ezgripper_offset_x} ${ezgripper_offset_y} ${ezgripper_offset_z}" rpy="0 0 0"/>
+<ezgripper_dual parent_link="base_link" prefix="only">
+  <origin xyz="${ezgripper_offset_x} ${ezgripper_offset_y} ${ezgripper_offset_z}" rpy="0 0 0"/>
 </ezgripper_dual>
 <link name="world"/>

File: ezgripper_driver/urdf/ezgripper_quad.urdf.xacro (robot description, xacro)
@@ -58,5 +58,6 @@
       <inertial>
         <mass value=".025"/>
-        <inertia ixx="0.01" ixy="0.0" ixz="0.0" iyy=".01" iyz="0.0" izz="0.01"/>
+        <pose>0.5 0.0 0 0.0 0.0 0.0</pose>
+        <inertia ixx="0.01" ixy="0.0" ixz="0.0" iyy="0.01" iyz="0.0" izz="0.01"/>
       </inertial>
     </link>
@@ -68,9 +69,22 @@
       <child link="${prefix}_ezgripper_finger_${postfix}"/>
       <origin xyz="0.1056 ${reflectY*0.03} ${reflectZ*0.03}" rpy="${1.5708 * reflectR} 0 3.14159"/>
-      <axis xyz="0 1 0"/>
+      <axis xyz="0 1 0">
+        <dynamics>
+          <spring_reference>0</spring_reference>
+          <spring_stiffness>1</spring_stiffness>
+        </dynamics>
+      </axis>
       <limit lower="-.27" upper="1.57075" effort="1" velocity="3.67"/>
       <xacro:if value="${mimic_test}">
            <mimic joint="${prefix}_ezgripper_knuckle_1"/>
       </xacro:if>
+      <physics>
+        <ode>
+          <limit>
+            <cfm>9.0</cfm>
+            <erp>1.0</erp>
+          </limit>
+        </ode>
+      </physics>
     </joint>
 </macro>

File: ezgripper_driver/urdf/ezgripper_quad_standalone.urdf.xacro (robot description, xacro)
@@ -6,5 +6,5 @@
 <xacro:include filename="$(find ezgripper_driver)/urdf/ezgripper_quad.urdf.xacro"/>
 <!-- Add the gripper -->
-<ezgripper_quad parent_link="base_link" prefix="1">
+<ezgripper_quad parent_link="base_link" prefix="only">
 <origin xyz="${ezgripper_offset_x} ${ezgripper_offset_y} ${ezgripper_offset_z}" rpy="0 0 0"/>
 </ezgripper_quad>

File: ezgripper_driver/urdf/ezgripper_urdf.urdf (robot description, URDF)
Before this commit: robot ezgripper_stand_alone, 3 links, 2 joints
Links:
- removed link 1_ezgripper_palm_link
- added link only_ezgripper_finger_1, mass .025; collision mesh filename=package://ezgripper_driver/meshes/collision/SAKE_Finger.stl; visual mesh filename=package://ezgripper_driver/meshes/visual/SAKE_Finger.stl
- added link only_ezgripper_finger_2, mass .025; collision mesh filename=package://ezgripper_driver/meshes/collision/SAKE_Finger.stl; visual mesh filename=package://ezgripper_driver/meshes/visual/SAKE_Finger.stl
- added link only_ezgripper_finger_3, mass .025; collision mesh filename=package://ezgripper_driver/meshes/collision/SAKE_Finger.stl; visual mesh filename=package://ezgripper_driver/meshes/visual/SAKE_Finger.stl
- added link only_ezgripper_finger_4, mass .025; collision mesh filename=package://ezgripper_driver/meshes/collision/SAKE_Finger.stl; visual mesh filename=package://ezgripper_driver/meshes/visual/SAKE_Finger.stl
- added link only_ezgripper_palm_link, mass .3; collision mesh filename=package://ezgripper_driver/meshes/collision/SAKE_Palm_Quad.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; visual mesh filename=package://ezgripper_driver/meshes/visual/SAKE_Palm_Quad.stl
Joints:
- removed joint 1_ezgripper_connect
- added joint only_ezgripper_connect: type fixed, parent base_link, child only_ezgripper_palm_link, origin xyz=0.049 0.0 0.2 rpy=-1.57 0 0, axis 0 0 0, limit lower=-1.57075 upper=0.25 effort=0 velocity=3.67
- added joint only_ezgripper_knuckle_1: type revolute, parent only_ezgripper_palm_link, child only_ezgripper_finger_1, origin xyz=0.1056 0.03 0.03 rpy=1.5708 0 3.14159, axis 0 1 0, limit lower=-.27 upper=1.57075 effort=1 velocity=3.67
- added joint only_ezgripper_knuckle_2: type revolute, parent only_ezgripper_palm_link, child only_ezgripper_finger_2, origin xyz=0.1056 -0.03 0.03 rpy=-1.5708 0 3.14159, axis 0 1 0, limit lower=-.27 upper=1.57075 effort=1 velocity=3.67, mimic joint=only_ezgripper_knuckle_1
- added joint only_ezgripper_knuckle_3: type revolute, parent only_ezgripper_palm_link, child only_ezgripper_finger_3, origin xyz=0.1056 0.03 -0.03 rpy=1.5708 0 3.14159, axis 0 1 0, limit lower=-.27 upper=1.57075 effort=1 velocity=3.67, mimic joint=only_ezgripper_knuckle_1
- added joint only_ezgripper_knuckle_4: type revolute, parent only_ezgripper_palm_link, child only_ezgripper_finger_4, origin xyz=0.1056 -0.03 -0.03 rpy=-1.5708 0 3.14159, axis 0 1 0, limit lower=-.27 upper=1.57075 effort=1 velocity=3.67, mimic joint=only_ezgripper_knuckle_1
