Commit message: saving temp progress

File: ezgripper_driver/urdf/dual.urdf (robot description, URDF)
Before this commit: robot ezgripper_stand_alone, 4 links, 3 joints
Joints:
- joint only_ezgripper_knuckle_2: mimic joint=ezgripper_knuckle_1 -> joint=only_ezgripper_knuckle_1

File: ezgripper_driver/urdf/ezgripper_dual.urdf.xacro (robot description, xacro)
@@ -67,6 +67,6 @@
       <axis xyz="0 1 0"/>
       <limit lower="-.27" upper="1.57075" effort="1" velocity="3.67"/>
-      <xacro:if value="${mimic_test}">
-           <mimic joint="ezgripper_knuckle_1"/>
+      <xacro:if value="${	_test}">
+           <mimic joint="${prefix}_ezgripper_knuckle_1"/>
       </xacro:if>
     </joint>

Commit message: working

File: ezgripper_driver/urdf/dual.urdf (robot description, URDF)
Before this commit: robot ezgripper_stand_alone, 4 links, 3 joints
Links:
- added link only_ezgripper_finger_tip_1, mass .025; collision mesh filename=package://ezgripper_driver/meshes/collision/SAKE_Finger_Lin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; visual mesh filename=package://ezgripper_driver/meshes/visual/SAKE_Finger_Link2.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
- added link only_ezgripper_finger_tip_2, mass .025; collision mesh filename=package://ezgripper_driver/meshes/collision/SAKE_Finger_Lin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; visual mesh filename=package://ezgripper_driver/meshes/visual/SAKE_Finger_Link2.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
- added link spring_force_calculation_link, mass .025; visual box size=0.01 0.01 0.01
- link only_ezgripper_finger_1: geometry collision mesh filename=package://ezgripper_driver/meshes/collision/SAKE_Finger_Lin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; visual mesh filename=package://ezgripper_driver/meshes/visual/SAKE_Finger_Link1.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
- link only_ezgripper_finger_2: geometry collision mesh filename=package://ezgripper_driver/meshes/collision/SAKE_Finger_Lin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; visual mesh filename=package://ezgripper_driver/meshes/visual/SAKE_Finger_Link1.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
Joints:
- added joint only_ezgripper_tip_joint_1: type revolute, parent only_ezgripper_finger_1, child only_ezgripper_finger_tip_1, origin xyz=-0.0655 0 0 rpy=0 0.31 0, axis 0 1 0, limit lower=-1.57 upper=0.31 effort=1 velocity=3.67
- added joint only_ezgripper_tip_joint_2: type revolute, parent only_ezgripper_finger_2, child only_ezgripper_finger_tip_2, origin xyz=-0.0655 0 0 rpy=0 0.31 0, axis 0 1 0, limit lower=-1.57 upper=0.31 effort=1 velocity=3.67
- added joint spring_force_calculation_joint: type revolute, parent only_ezgripper_palm_link, child spring_force_calculation_link, origin xyz=0 0 0.2 rpy=0 0 0, axis 0 1 0, limit lower=-.27 upper=1.57075 effort=1 velocity=3.67
- joint only_ezgripper_knuckle_2: mimic joint=only_ezgripper_knuckle_1 -> (none)

Commit message: working simulation with springs and grabbing objects

File: ezgripper_driver/urdf/dual.urdf (robot description, URDF)
Before this commit: robot ezgripper_stand_alone, 7 links, 6 joints
Links:
- link spring_force_calculation_link: mass .025 -> .05
Joints:
- joint spring_force_calculation_joint: origin xyz=0 0 0.2 rpy=0 0 0 -> xyz=0 0 0.063 rpy=0 0 0

Commit message: some working progress

File: ezgripper_driver/urdf/dual.urdf (robot description, URDF)
Before this commit: robot ezgripper_stand_alone, 7 links, 6 joints
Links:
- added link ezgripper_rx_ry; visual cylinder length=0.42 radius=0.02
- added link ezgripper_ry_rz; visual cylinder length=0.42 radius=0.02
- added link ezgripper_xy; visual cylinder length=0.42 radius=0.02
- added link ezgripper_yz; visual cylinder length=0.42 radius=0.02
- added link ezgripper_z_rx; visual cylinder length=0.42 radius=0.02
Joints:
- removed joint fixed
- added joint ezgripper_base_r_x: type revolute, parent ezgripper_z_rx, child ezgripper_rx_ry, origin xyz=0.0 0.0 0 rpy=0 0 0, axis 1 0 0, limit effort=100 velocity=3.67
- added joint ezgripper_base_r_y: type revolute, parent ezgripper_rx_ry, child ezgripper_ry_rz, origin xyz=0.0 0.0 0 rpy=0 0 0, axis 0 1 0, limit effort=100 velocity=3.67
- added joint ezgripper_base_r_z: type revolute, parent ezgripper_ry_rz, child only_ezgripper_palm_link, origin xyz=0.0 0.0 0 rpy=0 0 0, axis 0 0 1, limit effort=100 velocity=3.67
- added joint ezgripper_base_x: type prismatic, parent world, child ezgripper_xy, origin xyz=0.0 0.0 0 rpy=0 0 0, axis 1 0 0, limit effort=100 velocity=10
- added joint ezgripper_base_y: type prismatic, parent ezgripper_xy, child ezgripper_yz, origin xyz=0.0 0.0 0 rpy=0 0 0, axis 0 1 0, limit effort=100 velocity=10
- added joint ezgripper_base_z: type prismatic, parent ezgripper_yz, child ezgripper_z_rx, origin xyz=0.0 0.0 0 rpy=0 0 0, axis 0 0 1, limit effort=100 velocity=10

Commit message: semi working progress

File: ezgripper_driver/urdf/dual.urdf (robot description, URDF)
Before this commit: robot ezgripper_stand_alone, 12 links, 11 joints
Links:
- link ezgripper_rx_ry: mass None -> 1; geometry 
- link ezgripper_ry_rz: mass None -> 1; geometry 
- link ezgripper_xy: mass None -> 1; geometry 
- link ezgripper_yz: mass None -> 1; geometry 
- link ezgripper_z_rx: mass None -> 1; geometry 
Joints:
- joint ezgripper_base_r_z: origin xyz=0.0 0.0 0 rpy=0 0 0 -> xyz=0 0 0 rpy=0 0 0
- joint ezgripper_base_z: origin xyz=0.0 0.0 0 rpy=0 0 0 -> xyz=0.0 0.0 1 rpy=0 0 0

Commit message: grasp experiment with grasp orientation generator

File: ezgripper_driver/urdf/dual.urdf (robot description, URDF)
Before this commit: robot ezgripper_stand_alone, 7 links, 6 joints
Links:
- added link ezgripper_rx_ry, mass 1
- added link ezgripper_ry_rz, mass 1
- added link ezgripper_xy, mass 1
- added link ezgripper_yz, mass 1
- added link ezgripper_z_rx, mass 1
- added link only_ezgripper_kinect_link, mass 0.01; visual box size=0.01 0.02 0.01
Joints:
- removed joint fixed
- added joint base_rx: type revolute, parent ezgripper_z_rx, child ezgripper_rx_ry, origin xyz=0.0 0.0 0 rpy=0 0 0, axis 1 0 0, limit lower=-3.1415 upper=3.1415 effort=100 velocity=2
- added joint base_ry: type revolute, parent ezgripper_rx_ry, child ezgripper_ry_rz, origin xyz=0.0 0.0 0 rpy=0 0 0, axis 0 1 0, limit lower=-3.1415 upper=3.1415 effort=100 velocity=2
- added joint base_rz: type revolute, parent ezgripper_ry_rz, child only_ezgripper_palm_link, origin xyz=0 0 0 rpy=0 0 0, axis 0 0 1, limit lower=-3.1415 upper=3.1415 effort=100 velocity=2
- added joint base_x: type prismatic, parent world, child ezgripper_xy, origin xyz=0.0 0.0 0 rpy=0 0 0, axis 1 0 0, limit lower=-10 upper=10 effort=100 velocity=2
- added joint base_y: type prismatic, parent ezgripper_xy, child ezgripper_yz, origin xyz=0.0 0.0 0 rpy=0 0 0, axis 0 1 0, limit lower=-10 upper=10 effort=100 velocity=2
- added joint base_z: type prismatic, parent ezgripper_yz, child ezgripper_z_rx, origin xyz=0.0 0.0 0 rpy=0 0 0, axis 0 0 1, limit lower=-10 upper=10 effort=100 velocity=2
- added joint only_ezgripper_kinect_link: type fixed, parent only_ezgripper_palm_link, child only_ezgripper_kinect_link, origin xyz=0 0 0.17 rpy=0 0.5 0
- joint only_ezgripper_tip_joint_1: limit lower=-1.57 upper=0.31 effort=1 velocity=3.67 -> lower=-1.57 upper=0.26 effort=1 velocity=3.67; origin xyz=-0.0655 0 0 rpy=0 0.31 0 -> xyz=-0.0655 0 0 rpy=0 0.26 0
- joint only_ezgripper_tip_joint_2: limit lower=-1.57 upper=0.31 effort=1 velocity=3.67 -> lower=-1.57 upper=0.26 effort=1 velocity=3.67; origin xyz=-0.0655 0 0 rpy=0 0.31 0 -> xyz=-0.0655 0 0 rpy=0 0.26 0

Commit message: another progress save

File: ezgripper_driver/urdf/dual.urdf (robot description, URDF)
Before this commit: robot ezgripper_stand_alone, 13 links, 12 joints
Links:
- added link only_ezgripper_finger_inner_contact_1, mass 0.005; collision box size=0.033 0.025 0.004; visual box size=0.033 0.025 0.004
- added link only_ezgripper_finger_inner_contact_2, mass 0.005; collision box size=0.033 0.025 0.004; visual box size=0.033 0.025 0.004
- added link only_ezgripper_finger_tip_contact_1, mass 0.005; collision box size=0.06 0.025 0.004; visual box size=0.06 0.025 0.004
- added link only_ezgripper_finger_tip_contact_2, mass 0.005; collision box size=0.06 0.025 0.004; visual box size=0.06 0.025 0.004
Joints:
- added joint only_ezgripper_inner_contact_joint_1: type fixed, parent only_ezgripper_finger_1, child only_ezgripper_finger_inner_contact_1, origin xyz=-0.037 0 -0.014 rpy=0 0 0
- added joint only_ezgripper_inner_contact_joint_2: type fixed, parent only_ezgripper_finger_2, child only_ezgripper_finger_inner_contact_2, origin xyz=-0.037 0 -0.014 rpy=0 0 0
- added joint only_ezgripper_tip_contact_joint_1: type fixed, parent only_ezgripper_finger_tip_1, child only_ezgripper_finger_tip_contact_1, origin xyz=-0.043 0 -0.014 rpy=0 0 0
- added joint only_ezgripper_tip_contact_joint_2: type fixed, parent only_ezgripper_finger_tip_2, child only_ezgripper_finger_tip_contact_2, origin xyz=-0.043 0 -0.014 rpy=0 0 0
- joint only_ezgripper_tip_joint_1: limit lower=-1.57 upper=0.26 effort=1 velocity=3.67 -> lower=-1.57 upper=0.28 effort=1 velocity=3.67; origin xyz=-0.0655 0 0 rpy=0 0.26 0 -> xyz=-0.0655 0 0 rpy=0 0 0
- joint only_ezgripper_tip_joint_2: limit lower=-1.57 upper=0.26 effort=1 velocity=3.67 -> lower=-1.57 upper=0.28 effort=1 velocity=3.67; origin xyz=-0.0655 0 0 rpy=0 0.26 0 -> xyz=-0.0655 0 0 rpy=0 0 0
